File: kicad/sensor-hub.sch (KiCad schematic (older format))
At the start: 42 parts, among them J1 USB_B_Micro, J10 DHT22, J11 MQ_Sensors, J12 I2C-Si7021, J13 BG312L, J14 CC_DBG, J15 BT_DBG, J16 ZB_DBG, J17 CC_PWR, J5 ESP_TXD, J6 ESP_RXD, J7 DallasPullUp, J8 IRRecv/Dallas, J9 BH1750/Display, Q3 PN2222A, SW1 SW_Flash, U1 AP1117-33, U2 ESP-12F, U3 SZ1-CC2530, U5 CH330N

Commit message: WIP: v0.4 with pin order converter board
Signed-off-by: Zamir SUN <sztsian@gmail.com>
Parts:
- removed J10: DHT22, Connector_PinSocket_2.54mm:PinSocket_1x03_P2.54mm_Vertical, symbol Connector:Conn_01x03_Female
- removed J12: I2C-Si7021, Connector_PinSocket_2.54mm:PinSocket_1x04_P2.54mm_Vertical, symbol Connector:Conn_01x04_Female
- removed J7: DallasPullUp, Connector_PinHeader_2.54mm:PinHeader_1x02_P2.54mm_Vertical, symbol Connector:Conn_01x02_Male
- removed J8: IRRecv/Dallas, Connector_PinSocket_2.54mm:PinSocket_1x03_P2.54mm_Vertical, symbol Connector:Conn_01x03_Female
- added J17, J20, J7: Si7021, Connector_PinHeader_2.54mm:PinHeader_1x04_P2.54mm_Vertical, symbol Connector:Conn_01x04_Male
- added J18, J21: HDC1080, Connector_PinSocket_2.54mm:PinSocket_1x04_P2.54mm_Vertical, symbol Connector:Conn_01x04_Female
- added J19, J22, J9: SHT, Connector_PinSocket_2.54mm:PinSocket_1x04_P2.54mm_Vertical, symbol Connector:Conn_01x04_Female
- added J2: IO14/SHT, Connector_PinSocket_2.54mm:PinSocket_2x04_P2.54mm_Vertical, symbol Connector_Generic:Conn_02x04_Odd_Even
- added J3: HDC/Si7021, Connector_PinSocket_2.54mm:PinSocket_2x04_P2.54mm_Vertical, symbol Connector_Generic:Conn_02x04_Odd_Even
- added J4: IO12/SHT, Connector_PinSocket_2.54mm:PinSocket_2x04_P2.54mm_Vertical, symbol Connector_Generic:Conn_02x04_Odd_Even
- added J8: HTU21D, Connector_PinSocket_2.54mm:PinSocket_1x04_P2.54mm_Vertical, symbol Connector:Conn_01x04_Female
- added JP2: SJ_GPIO14, Jumper:SolderJumper-2_P1.3mm_Open_TrianglePad1.0x1.5mm, symbol Jumper:SolderJumper_2_Open
- added JP3: SJ_GPIO12, Jumper:SolderJumper-2_P1.3mm_Open_TrianglePad1.0x1.5mm, symbol Jumper:SolderJumper_2_Open
- added R1: 4.7k, Resistor_SMD:R_0603_1608Metric_Pad1.05x0.95mm_HandSolder, symbol Device:R_Small
- renumbered J9 to J10, J17 to J12
Connections:
- wire segments 62 -> 61

Commit message: Finalize v0.4 version without pin converter board
Signed-off-by: Zamir SUN <sztsian@gmail.com>
Parts:
- removed J17, J20, J7: Si7021, Connector_PinHeader_2.54mm:PinHeader_1x04_P2.54mm_Vertical, symbol Connector:Conn_01x04_Male
- removed J18, J21: HDC1080, Connector_PinSocket_2.54mm:PinSocket_1x04_P2.54mm_Vertical, symbol Connector:Conn_01x04_Female
- removed J19, J22, J9: SHT, Connector_PinSocket_2.54mm:PinSocket_1x04_P2.54mm_Vertical, symbol Connector:Conn_01x04_Female
- removed J8: HTU21D, Connector_PinSocket_2.54mm:PinSocket_1x04_P2.54mm_Vertical, symbol Connector:Conn_01x04_Female
- J1: symbol Connector:USB_B_Micro -> sensor-hub-rescue:USB_B_Micro-Connector
